File: 7SegmentDisplay_DualLine_NoDriver/8Inches/7SegmentDisplay_DualLine_NoDriver_8Inches_188/7SegmentDisplay_DualLine_NoDriver_8Inches_188.kicad_pcb (KiCad board)
At the start: 2 copper layers, 330.6 x 247 mm, 420 parts

Commit message: ADDED: 7SegmentDisplay DualLine without Driver
Other:
- board text added: "12"
- board text added: "A B C D E F G"
